File: eagle-schematics/main-board.sch (EAGLE design)
At the start: 0 parts

Commit message: Added EAGLE files
Parts:
- added 7.5V: POWER, SparkFun-Connectors:POWER_JACKSLT
- added ARDUINO: ARDUINO_PRO_MINI, SparkFun-Boards:ARDUINO_PRO_MINI
- added C1: 470uF, rcl:CPOL-EUB45181A
- added C2: 47uF, rcl:CPOL-EUB45181A
- added CLOSE, OPEN: MSWITCH, SparkFun-Switches:MOMENTARY-SWITCH-SPST-PTH-6.0MM
- added FUSE: 7.5V/0.5A, SparkFun-Fuses:PPTC_PTH
- added IR-REC: VS1838B, SparkFun-Sensors:BRM-2A18VERT
- added LIMIT: (no value), SparkFun-Connectors:CONN_03
- added PHOTO: PHOTOCELLPTH, SparkFun-Sensors:PHOTOCELLPTH
- added PWR_SW: (no value), SparkFun-Switches:SWITCH-SPDT-PTH-11.6X4.0MM
- added R1, R2: 1k, SparkFun-Resistors:1KOHM-HORIZ-1/4W-1%
- added R3: 15k, SparkFun-Resistors:RESISTORAXIAL-0.3
- added R4: 47, SparkFun-Resistors:RESISTORAXIAL-0.3
- added R5, R6, R7: 10k, SparkFun-Resistors:1KOHM-HORIZ-1/4W-1%
- added RGB-BLU, RGB-GRN, RGB-RED: 330, SparkFun-Resistors:RESISTORAXIAL-0.3
- added RGB-LED: DIFFUSE, autocurtain-components:5MMRGBLED
- added STEPPER: (no value), SparkFun-Connectors:CONN_05
- added TMP36: (no value), SparkFun-Sensors:TMP36GT9
- added ULN2003: ULN2003AN, uln-udn:ULN2003AN
Connections:
- new net 5V: ARDUINO.RAW, C1.+, CLOSE.1, FUSE.1, IR-REC.VCC, LIMIT.3, OPEN.1, PHOTO.P$2, PWR_SW.O, R3.1, R4.1, R7.2, TMP36.VCC, ULN2003.CD+
- new net A0: ARDUINO.A0, PHOTO.P$1, R5.2
- new net A1: ARDUINO.A1, IR-REC.OUT, R3.2
- new net A2: ARDUINO.A2, TMP36.VOUT
- new net AFTER: ARDUINO.RST@2, R7.1
- new net D10: ARDUINO.*10, ULN2003.I3
- new net D12: ARDUINO.12, ULN2003.I4
- new net D13: ARDUINO.13, LIMIT.2, R6.2
- new net D3: ARDUINO.*3, OPEN.2, R1.1
- new net D4: ARDUINO.4, CLOSE.2, R2.1
- new net D5: ARDUINO.*5, RGB-RED.1
- new net D6: ARDUINO.*6, RGB-BLU.1
- new net D7: ARDUINO.7, RGB-GRN.1
- new net D8: ARDUINO.8, ULN2003.I1
- new net D9: ARDUINO.*9, ULN2003.I2
- new net FUSE: FUSE.2, STEPPER.5
- new net GND: 7.5V.GND, 7.5V.GNDBREAK, ARDUINO.GND, ARDUINO.GND@2, C1.-, C2.-, IR-REC.GND, R1.2, R2.2, R5.1, R6.1, RGB-LED.GND, TMP36.GND, ULN2003.GND
- new net N$1: 7.5V.PWR, PWR_SW.P
- new net N$2: C2.+, R4.2
- new net N$3: RGB-BLU.2, RGB-LED.BLUE
- new net N$4: RGB-GRN.2, RGB-LED.GREEN
- new net N$5: STEPPER.1, ULN2003.O1
- new net N$6: STEPPER.2, ULN2003.O2
- new net N$7: STEPPER.3, ULN2003.O3
- new net N$8: STEPPER.4, ULN2003.O4
- new net N$9: RGB-LED.RED, RGB-RED.2
Other:
- note added: "Separated from board with cable package"

Commit message: Updated PCB design
Parts:
- added A3, A4, A5, A6, A7, D11, D2, RS, RX, TX, VC: LSP11, solpad:LSP11
Connections:
- new net N$10: A6.MP, ARDUINO.A6
- new net N$11: A7.MP, ARDUINO.A7
- new net N$12: A5.MP, ARDUINO.A5
- new net N$13: A4.MP, ARDUINO.A4
- new net N$14: A3.MP, ARDUINO.A3
- new net N$15: ARDUINO.VCC, VC.MP
- new net N$16: ARDUINO.2, D2.MP
- new net N$17: ARDUINO.RST, RS.MP
- new net N$18: ARDUINO.RXI, RX.MP
- new net N$19: ARDUINO.TXO, TX.MP
- new net N$20: ARDUINO.*11, D11.MP
Other:
- moved on the sheet: 7.5V, C1, PWR_SW, R7
